File: cpu_socket_expansion/pcb/cpu_socket_expansion.kicad_pcb (KiCad board)
At the start: 2 copper layers, 42.6 x 74.7 mm, 54 parts, among them M16 16MHz

Commit message: cpu_socket_expansion: Board that plugs into an Elk/Beeb CPU socket and allows FPGA daughterboards.
Parts:
- added R2: 10k, Resistors_SMD:R_0805_HandSoldering, B.Cu at (155.6, 110.5)
- added R3: 10k, Resistors_SMD:R_0805_HandSoldering, F.Cu at (156.6, 115.0)
- added R4: 10k, Resistors_SMD:R_0805_HandSoldering, F.Cu at (150.6, 65.0)
- added R5: 10k, Resistors_SMD:R_0805_HandSoldering, F.Cu at (151.1, 68.5)
- added R6: 10k, Resistors_SMD:R_0805_HandSoldering, F.Cu at (153.1, 68.5)
- moved staple_single5 2.27 mm to (154.3, 63.0)
- moved staple_single27 0.31 mm to (155.0, 107.2)
Routing:
- net 3V3: track 134.4 -> 145.5 mm
- net dbuf_nCE: track 43.9 -> 50.9 mm
- net ext_GP0: track 32.1 -> 35.5 mm
- net ext_GP2: track 30.7 -> 33.8 mm
- net ext_GP1: track 23.4 -> 26.2 mm
- net ext_GP3: track 21.0 -> 22.6 mm
- net ext_GP4: track 24.6 -> 25.6 mm
- net abuf_nCE: track 60.3 -> 61.2 mm
Other:
- board text added: "1"
- board text added: "<- GND/VPB"
- board text added: "Gap to allow for the two boards to connect to each other"
- board text added: "RF circuitry blocks us on the left"
- board text added: "avoid keyboard connector on Electron"
- board text added: "pp@myelin.nz cpu_socket_expansion For installation into an Electron or BBC B"
