File: master_updateable_megarom/pcb/master_updateable_megarom.kicad_pcb (KiCad board)
At the start: 2 copper layers, 36 x 49 mm, 25 parts

Commit message: master_updateable_megarom: Renamed JP1 and JP2 to JP0 and JP1
Connections:
- CPLD pad 19: cpld_JP2 -> cpld_JP1
- CPLD pad 22: cpld_JP1 -> cpld_JP0
- JP pad 2: cpld_JP1 -> cpld_JP0
- JP pad 3: cpld_JP2 -> cpld_JP1
Routing:
- net cpld_JP0: track 0.00 -> 24.5 mm, vias 0 -> 1
- net cpld_JP2: track 21.6 -> 0.00 mm, vias 1 -> 0
- net cpld_JP1: track 24.5 -> 21.6 mm
Changed lines of the file:
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@@
     (links 113)
     (no_connects 0)
-    (area 80 30 167.000001 107.000001)
+    (area 103.949999 42.949999 140.050001 92.050001)
     (thickness 1.6)
     (drawings 13)
@@
   (net 57 cpld_SS)
   (net 58 cpld_JP1)
-  (net 59 cpld_JP2)
+  (net 59 cpld_JP0)
   (net_class Default "This is the default net class."
     (clearance 0.1778)
@@
     (add_net bbc_A8)
     (add_net bbc_A9)
+    (add_net cpld_JP0)
     (add_net cpld_JP1)
-    (add_net cpld_JP2)
     (add_net cpld_MISO)
     (add_net cpld_MOSI)
@@
       (net 10 bbc_A12))
     (pad 19 smd rect (at -2.75 6 180) (size 0.25 2) (layers F.Cu F.Paste F.Mask)
-      (net 59 cpld_JP2))
+      (net 58 cpld_JP1))
     (pad 20 smd rect (at -2.25 6 180) (size 0.25 2) (layers F.Cu F.Paste F.Mask)
       (net 8 bbc_A15))
@@
       (net 2 GND))
     (pad 22 smd rect (at -1.25 6 180) (size 0.25 2) (layers F.Cu F.Paste F.Mask)
-      (net 58 cpld_JP1))
+      (net 59 cpld_JP0))
     (pad 23 smd rect (at -0.75 6 180) (size 0.25 2) (layers F.Cu F.Paste F.Mask)
       (net 30 bbc_A13))
@@
       (net 2 GND))
     (pad 2 thru_hole oval (at 0 2.54 90) (size 1.7 1.7) (drill 1) (layers *.Cu *.Mask)
+      (net 59 cpld_JP0))
+    (pad 3 thru_hole oval (at 0 5.08 90) (size 1.7 1.7) (drill 1) (layers *.Cu *.Mask)
       (net 58 cpld_JP1))
-    (pad 3 thru_hole oval (at 0 5.08 90) (size 1.7 1.7) (drill 1) (layers *.Cu *.Mask)
-      (net 59 cpld_JP2))
     (pad 4 thru_hole oval (at 0 7.62 90) (size 1.7 1.7) (drill 1) (layers *.Cu *.Mask)
       (net 3 5V))
@@
   (segment (start 112.83 53.01) (end 110.37 55.47) (width 0.1778) (layer B.Cu) (net 57))
   (segment (start 112.83 51.76) (end 112.83 53.01) (width 0.1778) (layer B.Cu) (net 57))
-  (segment (start 126.69 53.57) (end 129.23 53.57) (width 0.1778) (layer B.Cu) (net 58))
-  (segment (start 129.23 53.57) (end 130.51 52.29) (width 0.1778) (layer B.Cu) (net 58))
-  (segment (start 125.033299 51.913299) (end 126.69 53.57) (width 0.1778) (layer B.Cu) (net 58))
-  (segment (start 119.233299 52.876701) (end 120.196701 51.913299) (width 0.1778) (layer B.Cu) (net 58))
-  (segment (start 120.196701 51.913299) (end 125.033299 51.913299) (width 0.1778) (layer B.Cu) (net 58))
-  (segment (start 115.55764 55.68236) (end 118.363299 52.876701) (width 0.1778) (layer B.Cu) (net 58))
-  (segment (start 118.363299 52.876701) (end 119.233299 52.876701) (width 0.1778) (layer B.Cu) (net 58))
-  (segment (start 115.15236 55.68236) (end 115.55764 55.68236) (width 0.1778) (layer B.Cu) (net 58))
-  (segment (start 114.745961 55.275961) (end 115.15236 55.68236) (width 0.1778) (layer B.Cu) (net 58))
-  (segment (start 114.5 59.19409) (end 114.755212 58.938878) (width 0.1778) (layer F.Cu) (net 58))
-  (segment (start 114.755212 58.938878) (end 114.755212 58.292698) (width 0.1778) (layer F.Cu) (net 58))
-  (segment (start 114.4052 57.942686) (end 114.207624 57.942686) (width 0.1778) (layer F.Cu) (net 58))
-  (segment (start 114.5 60.2) (end 114.5 59.19409) (width 0.1778) (layer F.Cu) (net 58))
-  (segment (start 114.755212 58.292698) (end 114.4052 57.942686) (width 0.1778) (layer F.Cu) (net 58))
-  (segment (start 114.207624 57.942686) (end 113.983601 57.718663) (width 0.1778) (layer F.Cu) (net 58))
-  (segment (start 113.983601 57.718663) (end 113.983601 56.038321) (width 0.1778) (layer F.Cu) (net 58))
-  (segment (start 113.983601 56.038321) (end 114.339562 55.68236) (width 0.1778) (layer F.Cu) (net 58))
-  (segment (start 114.339562 55.68236) (end 114.745961 55.275961) (width 0.1778) (layer F.Cu) (net 58))
-  (via (at 114.745961 55.275961) (size 0.8128) (drill 0.3302) (layers F.Cu B.Cu) (net 58))
-  (segment (start 131.293299 54.046701) (end 132.200001 53.139999) (width 0.1778) (layer B.Cu) (net 59))
-  (segment (start 132.200001 53.139999) (end 133.05 52.29) (width 0.1778) (layer B.Cu) (net 59))
-  (segment (start 120.041377 54.046701) (end 131.293299 54.046701) (width 0.1778) (layer B.Cu) (net 59))
-  (segment (start 117.507525 56.580553) (end 120.041377 54.046701) (width 0.1778) (layer B.Cu) (net 59))
-  (segment (start 117.101126 56.986952) (end 117.507525 56.580553) (width 0.1778) (layer F.Cu) (net 59))
-  (segment (start 116 58.399248) (end 117.101126 57.298122) (width 0.1778) (layer F.Cu) (net 59))
-  (segment (start 116 60.2) (end 116 58.399248) (width 0.1778) (layer F.Cu) (net 59))
-  (segment (start 117.101126 57.298122) (end 117.101126 56.986952) (width 0.1778) (layer F.Cu) (net 59))
-  (via (at 117.507525 56.580553) (size 0.8128) (drill 0.3302) (layers F.Cu B.Cu) (net 59))
+  (segment (start 131.293299 54.046701) (end 132.200001 53.139999) (width 0.1778) (layer B.Cu) (net 58))
+  (segment (start 132.200001 53.139999) (end 133.05 52.29) (width 0.1778) (layer B.Cu) (net 58))
+  (segment (start 120.041377 54.046701) (end 131.293299 54.046701) (width 0.1778) (layer B.Cu) (net 58))
+  (segment (start 117.507525 56.580553) (end 120.041377 54.046701) (width 0.1778) (layer B.Cu) (net 58))
+  (segment (start 117.101126 56.986952) (end 117.507525 56.580553) (width 0.1778) (layer F.Cu) (net 58))
+  (segment (start 116 58.399248) (end 117.101126 57.298122) (width 0.1778) (layer F.Cu) (net 58))
+  (segment (start 116 60.2) (end 116 58.399248) (width 0.1778) (layer F.Cu) (net 58))
+  (segment (start 117.101126 57.298122) (end 117.101126 56.986952) (width 0.1778) (layer F.Cu) (net 58))
+  (via (at 117.507525 56.580553) (size 0.8128) (drill 0.3302) (layers F.Cu B.Cu) (net 58))
+  (segment (start 126.69 53.57) (end 129.23 53.57) (width 0.1778) (layer B.Cu) (net 59))
+  (segment (start 129.23 53.57) (end 130.51 52.29) (width 0.1778) (layer B.Cu) (net 59))
+  (segment (start 125.033299 51.913299) (end 126.69 53.57) (width 0.1778) (layer B.Cu) (net 59))
+  (segment (start 119.233299 52.876701) (end 120.196701 51.913299) (width 0.1778) (layer B.Cu) (net 59))
+  (segment (start 120.196701 51.913299) (end 125.033299 51.913299) (width 0.1778) (layer B.Cu) (net 59))
+  (segment (start 115.55764 55.68236) (end 118.363299 52.876701) (width 0.1778) (layer B.Cu) (net 59))
+  (segment (start 118.363299 52.876701) (end 119.233299 52.876701) (width 0.1778) (layer B.Cu) (net 59))
+  (segment (start 115.15236 55.68236) (end 115.55764 55.68236) (width 0.1778) (layer B.Cu) (net 59))
+  (segment (start 114.745961 55.275961) (end 115.15236 55.68236) (width 0.1778) (layer B.Cu) (net 59))
+  (segment (start 114.5 59.19409) (end 114.755212 58.938878) (width 0.1778) (layer F.Cu) (net 59))
+  (segment (start 114.755212 58.938878) (end 114.755212 58.292698) (width 0.1778) (layer F.Cu) (net 59))
+  (segment (start 114.4052 57.942686) (end 114.207624 57.942686) (width 0.1778) (layer F.Cu) (net 59))
+  (segment (start 114.5 60.2) (end 114.5 59.19409) (width 0.1778) (layer F.Cu) (net 59))
+  (segment (start 114.755212 58.292698) (end 114.4052 57.942686) (width 0.1778) (layer F.Cu) (net 59))
+  (segment (start 114.207624 57.942686) (end 113.983601 57.718663) (width 0.1778) (layer F.Cu) (net 59))
+  (segment (start 113.983601 57.718663) (end 113.983601 56.038321) (width 0.1778) (layer F.Cu) (net 59))
+  (segment (start 113.983601 56.038321) (end 114.339562 55.68236) (width 0.1778) (layer F.Cu) (net 59))
+  (segment (start 114.339562 55.68236) (end 114.745961 55.275961) (width 0.1778) (layer F.Cu) (net 59))
+  (via (at 114.745961 55.275961) (size 0.8128) (drill 0.3302) (layers F.Cu B.Cu) (net 59))
   (zone (net 2) (net_name GND) (layer F.Cu) (hatch edge 0.508)
     (connect_pads (clearance 0.254))
