File: expansion_minispartan_breakout/pcb/acorn-electron-expansion.kicad_pcb (KiCad board)
At the start: 2 copper layers, 100 x 100 mm, 19 parts, among them P1 Acorn Electron Expansion Conn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, P2 CONN_02X24, P3 5V / 5V0, U1 74hct125d, U2 74LVC245 D0-7, U3 74LVC245 A0-7, U4 74LVC245 A8-15, U5 74LVC245, U6 scarab_mini_spartan_6_lx25

Commit message: Updates to expansion_minispartan_breakout to allow the FPGA to drive the bus
Parts:
- added R6: 10k, Resistors_SMD:R_0805_HandSoldering, F.Cu at (166.2, 75.8)
- added R7: 10k, Resistors_SMD:R_0805_HandSoldering, F.Cu at (136.6, 132.8)
- moved R4 16.2 mm to (145.7, 97.8), turned to 90 degrees
- moved R5 13.5 mm to (141.8, 97.8), turned to 90 degrees
- moved R3 13.5 mm to (115.2, 97.8)
- moved R1 13.3 mm to (117.7, 97.8)
- moved R2 3.26 mm to (115.2, 87.8), turned to 270 degrees
Connections:
- net /nASSERT_nRDY renamed /nDEASSERT_RDY
- net /nRDY renamed /RDY
- net /nRDY_3V renamed /RDY_3V
- U1 pad 11: Net-(U1-Pad11) -> /RnW
- U1 pad 12: /GND -> /RnW_OUT_3V
- U1 pad 13: /5V -> /RnW_nOE
- U3 pad 1: /3V3 -> /A_DIR
- U4 pad 1: /3V3 -> /A_DIR
- U5 pad 11: Net-(U5-Pad11) -> /nNMI_3V
- U5 pad 12: Net-(U5-Pad12) -> /nIRQ_3V
- U5 pad 8: /GND -> /nIRQ
- U5 pad 9: /GND -> /nNMI
- U6 pad C11: Net-(U6-PadC11) -> /A_DIR
- U6 pad D1: (no net) -> Net-(U6-PadD1)
- U6 pad D3: Net-(U6-PadD3) -> /RnW_OUT_3V
- U6 pad E1: (no net) -> /RnW_nOE
- U6 pad E3: Net-(U6-PadE3) -> /nNMI_3V
- U6 pad E5: Net-(U6-PadE5) -> /nIRQ_3V
- U6 pad F1: (no net) -> Net-(U6-PadF1)
Routing:
- net /nIRQ_3V: track 0.00 -> 69.0 mm, vias 0 -> 2
- net /RnW_nOE: track 0.00 -> 67.6 mm, vias 0 -> 2
- net /nNMI_3V: track 0.00 -> 66.4 mm, vias 0 -> 2
- net /RnW_OUT_3V: track 0.00 -> 66.0 mm, vias 0 -> 2
- net /A_DIR: track 0.00 -> 38.1 mm, vias 0 -> 1
- net /RnW: track 19.0 -> 42.3 mm, vias 0 -> 2
- net /nIRQ: track 43.6 -> 57.4 mm, vias 0 -> 2
- net /GND: track 79.9 -> 90.3 mm, vias 12 -> 11
- net /nNMI: track 36.3 -> 45.0 mm, vias 0 -> 1
- net /5V: track 72.7 -> 68.0 mm
- net /DATA_nOE: track 14.8 -> 19.0 mm
- net /RDY: track 65.7 -> 62.9 mm
- net /DATA_READ: track 23.4 -> 26.1 mm
- net /nASSERT_nIRQ: track 20.5 -> 22.8 mm, vias 2 -> 1
- net /nASSERT_nNMI: track 23.6 -> 25.0 mm, vias 2 -> 1
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Other:
- board text added: "### r1 -> r2 changes ### - RnW added to U1, P2, U6: RnW: U1.11, P2.17 RnW_OUT_3V: U1.12, U6.D3 RnW_nOE: U1.13, U6.E1 R7: 10k pullup on RnW_nOE to 3V3 - A_DIR added: U6.C11, U3.1, U4.1 R6: 10k pullup on A_DIR to 3V3 - nIRQ/nNMI added to U5 and FPGA nIRQ: U5.8, U6.E5 nNMI: U5.9, U6.E3"
- board text added: "Acorn Electron AN15 Expansion Connector debug / breakout board r2 Design by Phillip Pearson <pp@myelin.co.nz> Copyright 2017 Google Inc"
- board text added: "Acorn Electron AN15 Expansion Connector debug / breakout board r2 Design by Phillip Pearson <pp@myelin.co.nz> Copyright 2017 Google Inc github.com/google/myelin-acorn-electron-hardware/ expansion_minispartan_breakout"
- board text removed: "Acorn Electron AN15 Expansion Connector debug / breakout board Design by Phillip Pearson <pp@myelin.co.nz> Copyright 2017 Google Inc"
- board text removed: "Acorn Electron AN15 Expansion Connector debug / breakout board Design by Phillip Pearson <pp@myelin.co.nz> Copyright 2017 Google Inc github.com/google/myelin-acorn-electron-hardware/ expansion_minispartan_breakout"
