File: atsamd21_usb_host/pcb/atsamd21_usb.kicad_pcb (KiCad board)
At the start: 2 copper layers, 34 x 34.7 mm, 40 parts, among them U1 MCP1700T-3302E/MB, X1 MC146 32768Hz

Commit message: Tested atsamd21 board, and it works
Other:
- board text added: "atsamd21_usb_host r2 Phillip Pearson 2017"
- board text removed: "atsamd21_usb_host Phillip Pearson 2017"
Changed lines of the file:
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@@
     (links 97)
     (no_connects 0)
-    (area 165.749999 130.249999 199.850001 165.050001)
+    (area 131.479999 118.62 231.680001 169.870001)
     (thickness 1.6)
     (drawings 15)
@@
     )
   )
-  (module myelin-kicad:micro_usb_b_smd_molex (layer B.Cu)
-    (at 190.18 162.98 180)
-    (descr "Molex SD-105017-001 bottom mount micro USB socket")
-    (fp_text reference USB (at 0 -1 180) (layer B.SilkS)
-      (effects (font (size 1 1) (thickness 0.15)) (justify mirror))
-    )
-    (fp_text value usb (at 0 4 180) (layer B.SilkS)
-      (effects (font (size 1 1) (thickness 0.15)) (justify mirror))
-    )
-    (fp_line (start -4 3) (end 4 3) (layer B.SilkS) (width 0.15))
-    (fp_line (start -4 3) (end -4 -2) (layer B.SilkS) (width 0.15))
-    (fp_line (start -4 -2) (end 4 -2) (layer B.SilkS) (width 0.15))
-    (fp_line (start 4 3) (end 4 -2) (layer B.SilkS) (width 0.15))
-    (fp_line (start -4 -2.7) (end -3 -2.7) (layer B.SilkS) (width 0.15))
-    (fp_line (start 3 -2.7) (end 4 -2.7) (layer B.SilkS) (width 0.15))
-    (fp_text user V (at -1.3 0.65 180) (layer B.SilkS)
-      (effects (font (size 0.7 0.7) (thickness 0.15)) (justify mirror))
-    )
-    (fp_text user - (at -0.65 0.65 180) (layer B.SilkS)
-      (effects (font (size 0.7 0.7) (thickness 0.15)) (justify mirror))
-    )
-    (fp_text user + (at 0 0.65 180) (layer B.SilkS)
-      (effects (font (size 0.7 0.7) (thickness 0.15)) (justify mirror))
-    )
-    (fp_text user I (at 0.65 0.65 180) (layer B.SilkS)
-      (effects (font (size 0.7 0.7) (thickness 0.15)) (justify mirror))
-    )
-    (fp_text user G (at 1.3 0.65 180) (layer B.SilkS)
-      (effects (font (size 0.7 0.7) (thickness 0.15)) (justify mirror))
-    )
-    (pad 1 smd rect (at -1.3 2.15 180) (size 0.4 1.35) (layers B.Cu B.Paste B.Mask)
-      (net 2 5V))
-    (pad 2 smd rect (at -0.65 2.15 180) (size 0.4 1.35) (layers B.Cu B.Paste B.Mask)
-      (net 12 USBDM))
-    (pad 3 smd rect (at 0 2.15 180) (size 0.4 1.35) (layers B.Cu B.Paste B.Mask)
-      (net 13 USBDP))
-    (pad 4 smd rect (at 0.65 2.15 180) (size 0.4 1.35) (layers B.Cu B.Paste B.Mask)
-      (net 14 USB_ID))
-    (pad 5 smd rect (at 1.3 2.15 180) (size 0.4 1.35) (layers B.Cu B.Paste B.Mask)
-      (net 1 GND))
-    (pad P0 thru_hole circle (at -2.5 2.15 180) (size 1.45 1.45) (drill 0.85) (layers *.Cu *.Mask))
-    (pad P1 thru_hole circle (at 2.5 2.15 180) (size 1.45 1.45) (drill 0.85) (layers *.Cu *.Mask))
-    (pad M0 thru_hole circle (at -3.5 -0.55 180) (size 1.9 1.9) (drill 1.3) (layers *.Cu *.Mask))
-    (pad M1 thru_hole circle (at 3.5 -0.55 180) (size 1.9 1.9) (drill 1.3) (layers *.Cu *.Mask))
-  )
   (module Capacitors_SMD:C_0805_HandSoldering (layer F.Cu)
     (at 184.24 138.59)
@@
     )
   )
+  (module myelin-kicad:micro_usb_b_smd_molex (layer B.Cu)
+    (at 190.18 162.98 180)
+    (descr "Molex SD-105017-001 bottom mount micro USB socket")
+    (fp_text reference USB (at 0 -1 180) (layer B.SilkS)
+      (effects (font (size 1 1) (thickness 0.15)) (justify mirror))
+    )
+    (fp_text value usb (at 0 4 180) (layer B.SilkS)
+      (effects (font (size 1 1) (thickness 0.15)) (justify mirror))
+    )
+    (fp_line (start -4 3) (end 4 3) (layer B.SilkS) (width 0.15))
+    (fp_line (start -4 3) (end -4 -2) (layer B.SilkS) (width 0.15))
+    (fp_line (start -4 -2) (end 4 -2) (layer B.SilkS) (width 0.15))
+    (fp_line (start 4 3) (end 4 -2) (layer B.SilkS) (width 0.15))
+    (fp_line (start -4 -2.7) (end -3 -2.7) (layer B.SilkS) (width 0.15))
+    (fp_line (start 3 -2.7) (end 4 -2.7) (layer B.SilkS) (width 0.15))
+    (fp_text user V (at -1.3 0.65 180) (layer B.SilkS)
+      (effects (font (size 0.7 0.7) (thickness 0.15)) (justify mirror))
+    )
+    (fp_text user - (at -0.65 0.65 180) (layer B.SilkS)
+      (effects (font (size 0.7 0.7) (thickness 0.15)) (justify mirror))
+    )
+    (fp_text user + (at 0 0.65 180) (layer B.SilkS)
+      (effects (font (size 0.7 0.7) (thickness 0.15)) (justify mirror))
+    )
+    (fp_text user I (at 0.65 0.65 180) (layer B.SilkS)
+      (effects (font (size 0.7 0.7) (thickness 0.15)) (justify mirror))
+    )
+    (fp_text user G (at 1.3 0.65 180) (layer B.SilkS)
+      (effects (font (size 0.7 0.7) (thickness 0.15)) (justify mirror))
+    )
+    (pad 1 smd rect (at -1.3 2.4 180) (size 0.4 1.85) (layers B.Cu B.Paste B.Mask)
+      (net 2 5V))
+    (pad 2 smd rect (at -0.65 2.4 180) (size 0.4 1.85) (layers B.Cu B.Paste B.Mask)
+      (net 12 USBDM))
+    (pad 3 smd rect (at 0 2.4 180) (size 0.4 1.85) (layers B.Cu B.Paste B.Mask)
+      (net 13 USBDP))
+    (pad 4 smd rect (at 0.65 2.4 180) (size 0.4 1.85) (layers B.Cu B.Paste B.Mask)
+      (net 14 USB_ID))
+    (pad 5 smd rect (at 1.3 2.4 180) (size 0.4 1.85) (layers B.Cu B.Paste B.Mask)
+      (net 1 GND))
+    (pad P0 thru_hole circle (at -2.5 2.15 180) (size 1.45 1.45) (drill 0.85) (layers *.Cu *.Mask))
+    (pad P1 thru_hole circle (at 2.5 2.15 180) (size 1.45 1.45) (drill 0.85) (layers *.Cu *.Mask))
+    (pad M0 thru_hole circle (at -3.5 -0.55 180) (size 1.9 1.9) (drill 1.3) (layers *.Cu *.Mask))
+    (pad M1 thru_hole circle (at 3.5 -0.55 180) (size 1.9 1.9) (drill 1.3) (layers *.Cu *.Mask))
+  )
   (gr_text 1 (at 188.32 137.03) (layer F.SilkS)
     (effects (font (size 1 1) (thickness 0.15)))
@@
     (effects (font (size 1 1) (thickness 0.15)) (justify left mirror))
   )
-  (gr_text "atsamd21_usb_host\nPhillip Pearson 2017" (at 184.1 132.69) (layer F.SilkS)
+  (gr_text "atsamd21_usb_host r2\nPhillip Pearson 2017" (at 184.1 132.69) (layer F.SilkS)
     (effects (font (size 1 1) (thickness 0.15)))
   )
