File: bbc_power_distribution/pcb/bbc_power.kicad_pcb (KiCad board)
At the start: 2 copper layers, 34 x 19 mm, 20 parts, among them M1 hole, M2 hole, P1 5V, P2 5V, P3 5V, P4 GND, P5 GND, P6 GND, P7 -5V, U1 Charge pump

Commit message: bbc_power_distribution is ready to go
Parts:
- EXTGND: value gnd -> 0v
- moved M2 1.74 mm to (147.6, 94.5)
- moved M1 0.83 mm to (147.6, 88.5)
Other:
- board text added: "bbc_power_distribution (C) 2017 Google LLC"
- board text added: "http:// myelin.nz/ acorn/ bbcpwr"
- board text removed: "bbc_power_distribution Phillip Pearson 2017"
- board text removed: "github.com/ google/ myelin- acorn- electron- hardware"
Changed lines of the file:
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@@
   )
   (setup
-    (last_trace_width 0.508)
+    (last_trace_width 0.1778)
     (user_trace_width 0.254)
     (user_trace_width 0.508)
@@
     (user_trace_width 1.27)
     (trace_clearance 0.1778)
-    (zone_clearance 0.508)
+    (zone_clearance 0.254)
     (zone_45_only no)
     (trace_min 0.1778)
@@
     )
   )
-  (module myelin-kicad:micro_usb_b_smd_molex (layer F.Cu)
-    (at 118 99.94 270)
-    (descr "Molex SD-105017-001 bottom mount micro USB socket")
-    (fp_text reference USB (at 0 1 270) (layer F.SilkS)
-      (effects (font (size 1 1) (thickness 0.15)))
-    )
-    (fp_text value usb (at 7.64 -0.44 270) (layer F.SilkS) hide
-      (effects (font (size 1 1) (thickness 0.15)))
-    )
-    (fp_line (start -4 -3) (end 4 -3) (layer F.SilkS) (width 0.15))
-    (fp_line (start -4 -3) (end -4 2) (layer F.SilkS) (width 0.15))
-    (fp_line (start -4 2) (end 4 2) (layer F.SilkS) (width 0.15))
-    (fp_line (start 4 -3) (end 4 2) (layer F.SilkS) (width 0.15))
-    (fp_line (start -4 2.7) (end -3 2.7) (layer F.SilkS) (width 0.15))
-    (fp_line (start 3 2.7) (end 4 2.7) (layer F.SilkS) (width 0.15))
-    (fp_text user V (at -1.3 -0.65 270) (layer F.SilkS)
-      (effects (font (size 0.7 0.7) (thickness 0.15)))
-    )
-    (fp_text user - (at -0.65 -0.65 270) (layer F.SilkS)
-      (effects (font (size 0.7 0.7) (thickness 0.15)))
-    )
-    (fp_text user + (at 0 -0.65 270) (layer F.SilkS)
-      (effects (font (size 0.7 0.7) (thickness 0.15)))
-    )
-    (fp_text user I (at 0.65 -0.65 270) (layer F.SilkS)
-      (effects (font (size 0.7 0.7) (thickness 0.15)))
-    )
-    (fp_text user G (at 1.3 -0.65 270) (layer F.SilkS)
-      (effects (font (size 0.7 0.7) (thickness 0.15)))
-    )
-    (pad 1 smd rect (at -1.3 -2.15 270) (size 0.4 1.35) (layers F.Cu F.Paste F.Mask)
-      (net 1 5V))
-    (pad 2 smd rect (at -0.65 -2.15 270) (size 0.4 1.35) (layers F.Cu F.Paste F.Mask))
-    (pad 3 smd rect (at 0 -2.15 270) (size 0.4 1.35) (layers F.Cu F.Paste F.Mask))
-    (pad 4 smd rect (at 0.65 -2.15 270) (size 0.4 1.35) (layers F.Cu F.Paste F.Mask))
-    (pad 5 smd rect (at 1.3 -2.15 270) (size 0.4 1.35) (layers F.Cu F.Paste F.Mask)
-      (net 2 GND))
-    (pad P0 thru_hole circle (at -2.5 -2.15 270) (size 1.45 1.45) (drill 0.85) (layers *.Cu *.Mask))
-    (pad P1 thru_hole circle (at 2.5 -2.15 270) (size 1.45 1.45) (drill 0.85) (layers *.Cu *.Mask))
-    (pad M0 thru_hole circle (at -3.5 0.55 270) (size 1.9 1.9) (drill 1.3) (layers *.Cu *.Mask))
-    (pad M1 thru_hole circle (at 3.5 0.55 270) (size 1.9 1.9) (drill 1.3) (layers *.Cu *.Mask))
-  )
   (module myelin-kicad:dc10a_barrel_jack (layer F.Cu)
     (at 126.89 89.95 180)
@@
   )
   (module myelin-kicad:pin_100_120mil (layer F.Cu)
-    (at 147.38 87.71)
+    (at 147.58 88.52)
     (fp_text reference M1 (at 6.17 -1.25) (layer F.SilkS) hide
       (effects (font (size 1 1) (thickness 0.15)))
@@
   )
   (module myelin-kicad:pin_100_120mil (layer F.Cu)
-    (at 147.38 92.79)
+    (at 147.58 94.52)
     (fp_text reference M2 (at 5.72 -2.71) (layer F.SilkS) hide
       (effects (font (size 1 1) (thickness 0.15)))
@@
       (effects (font (size 1 1) (thickness 0.15)))
     )
-    (fp_text value -5V (at 1.27 0) (layer F.SilkS)
+    (fp_text value -5V (at 0.11 1.45) (layer F.SilkS)
       (effects (font (size 1 1) (thickness 0.15)))
     )
@@
       (effects (font (size 1 1) (thickness 0.15)))
     )
-    (fp_text value gnd (at -0.01 15.78 360) (layer F.SilkS)
+    (fp_text value 0v (at 0.19 15.41 360) (layer F.SilkS)
       (effects (font (size 1 1) (thickness 0.15)))
     )
@@
     )
   )
-  (gr_text "bbc_power_distribution\nPhillip Pearson 2017" (at 137.29 94.72) (layer B.SilkS)
+  (module myelin-kicad:micro_usb_b_smd_molex (layer F.Cu)
+    (at 118 99.94 270)
+    (descr "Molex SD-105017-001 bottom mount micro USB socket")
+    (fp_text reference USB (at 0 1 270) (layer F.SilkS)
+      (effects (font (size 1 1) (thickness 0.15)))
+    )
+    (fp_text value usb (at 0 -4 270) (layer F.SilkS) hide
+      (effects (font (size 1 1) (thickness 0.15)))
+    )
+    (fp_line (start -4 -3) (end 4 -3) (layer F.SilkS) (width 0.15))
+    (fp_line (start -4 -3) (end -4 2) (layer F.SilkS) (width 0.15))
+    (fp_line (start -4 2) (end 4 2) (layer F.SilkS) (width 0.15))
+    (fp_line (start 4 -3) (end 4 2) (layer F.SilkS) (width 0.15))
+    (fp_line (start -4 2.7) (end -3 2.7) (layer F.SilkS) (width 0.15))
+    (fp_line (start 3 2.7) (end 4 2.7) (layer F.SilkS) (width 0.15))
+    (fp_text user V (at -1.3 -0.65 270) (layer F.SilkS)
+      (effects (font (size 0.7 0.7) (thickness 0.15)))
+    )
+    (fp_text user - (at -0.65 -0.65 270) (layer F.SilkS)
+      (effects (font (size 0.7 0.7) (thickness 0.15)))
+    )
+    (fp_text user + (at 0 -0.65 270) (layer F.SilkS)
+      (effects (font (size 0.7 0.7) (thickness 0.15)))
+    )
+    (fp_text user I (at 0.65 -0.65 270) (layer F.SilkS)
+      (effects (font (size 0.7 0.7) (thickness 0.15)))
+    )
+    (fp_text user G (at 1.3 -0.65 270) (layer F.SilkS)
+      (effects (font (size 0.7 0.7) (thickness 0.15)))
+    )
+    (pad 1 smd rect (at -1.3 -2.4 270) (size 0.4 1.85) (layers F.Cu F.Paste F.Mask)
+      (net 1 5V))
+    (pad 2 smd rect (at -0.65 -2.4 270) (size 0.4 1.85) (layers F.Cu F.Paste F.Mask))
+    (pad 3 smd rect (at 0 -2.4 270) (size 0.4 1.85) (layers F.Cu F.Paste F.Mask))
+    (pad 4 smd rect (at 0.65 -2.4 270) (size 0.4 1.85) (layers F.Cu F.Paste F.Mask))
+    (pad 5 smd rect (at 1.3 -2.4 270) (size 0.4 1.85) (layers F.Cu F.Paste F.Mask)
+      (net 2 GND))
+    (pad P0 thru_hole circle (at -2.5 -2.15 270) (size 1.45 1.45) (drill 0.85) (layers *.Cu *.Mask))
+    (pad P1 thru_hole circle (at 2.5 -2.15 270) (size 1.45 1.45) (drill 0.85) (layers *.Cu *.Mask))
+    (pad M0 thru_hole circle (at -3.5 0.55 270) (size 1.9 1.9) (drill 1.3) (layers *.Cu *.Mask))
+    (pad M1 thru_hole circle (at 3.5 0.55 270) (size 1.9 1.9) (drill 1.3) (layers *.Cu *.Mask))
+  )
+  (gr_text "bbc_power_distribution\n(C) 2017 Google LLC" (at 137.29 94.72) (layer B.SilkS)
     (effects (font (size 1 1) (thickness 0.2)) (justify mirror))
   )
-  (gr_text "github.com/\ngoogle/\nmyelin-\nacorn-\nelectron-\nhardware" (at 148.38 100.46) (layer B.SilkS)
+  (gr_text "http://\nmyelin.nz/\nacorn/\nbbcpwr" (at 147.91 101.54) (layer B.SilkS)
     (effects (font (size 0.75 0.75) (thickness 0.1875)) (justify left mirror))
   )
@@
   (gr_line (start 150 86) (end 150 105) (layer Edge.Cuts) (width 0.1))
   (gr_line (start 116 86) (end 150 86) (layer Edge.Cuts) (width 0.1))
+  (segment (start 120.15 98.64) (end 121.29 98.64) (width 0.508) (layer F.Cu) (net 1))
+  (segment (start 121.63 98.3) (end 121.63 95.687766) (width 0.508) (layer F.Cu) (net 1))
+  (segment (start 121.29 98.64) (end 121.63 98.3) (width 0.508) (layer F.Cu) (net 1))
+  (segment (start 121.63 95.687766) (end 127.367766 89.95) (width 0.508) (layer F.Cu) (net 1))
+  (segment (start 127.367766 89.95) (end 129.99 89.95) (width 0.508) (layer F.Cu) (net 1))
   (segment (start 138.33 98.25) (end 139.688 98.25) (width 0.508) (layer F.Cu) (net 1))
   (segment (start 139.688 98.25) (end 140.968 99.53) (width 0.508) (layer F.Cu) (net 1))
   (segment (start 140.968 99.53) (end 141.93 99.53) (width 0.508) (layer F.Cu) (net 1))
-  (segment (start 120.15 98.64) (end 120.625 98.64) (width 0.508) (layer F.Cu) (net 1))
-  (segment (start 120.625 98.64) (end 121.63 97.635) (width 0.508) (layer F.Cu) (net 1))
-  (segment (start 121.63 97.635) (end 121.63 95.687766) (width 0.508) (layer F.Cu) (net 1))
-  (segment (start 127.367766 89.95) (end 129.99 89.95) (width 0.508) (layer F.Cu) (net 1))
-  (segment (start 121.63 95.687766) (end 127.367766 89.95) (width 0.508) (layer F.Cu) (net 1))
   (segment (start 141.93 99.53) (end 141.93 97.56) (width 0.508) (layer F.Cu) (net 1))
   (segment (start 141.93 97.56) (end 142.09 97.4) (width 0.508) (layer F.Cu) (net 1))
@@
   (segment (start 146.762 103.448) (end 147.92 102.29) (width 0.508) (layer F.Cu) (net 3))
   (segment (start 147.92 102.29) (end 147.92 102.19) (width 0.508) (layer F.Cu) (net 3))
-  (segment (start 143.83 102.23) (end 145.87 102.23) (width 0.1778) (layer F.Cu) (net 4))
-  (segment (start 145.87 102.23) (end 145.88 102.24) (width 0.1778) (layer F.Cu) (net 4))
-  (segment (start 143.83 99.53) (end 145.87 99.53) (width 0.1778) (layer F.Cu) (net 5))
-  (segment (start 145.87 99.53) (end 145.88 99.54) (width 0.1778) (layer F.Cu) (net 5))
+  (segment (start 143.83 102.23) (end 145.87 102.23) (width 0.508) (layer F.Cu) (net 4))
+  (segment (start 145.87 102.23) (end 145.88 102.24) (width 0.508) (layer F.Cu) (net 4))
+  (segment (start 143.83 99.53) (end 145.87 99.53) (width 0.508) (layer F.Cu) (net 5))
+  (segment (start 145.87 99.53) (end 145.88 99.54) (width 0.508) (layer F.Cu) (net 5))
   (segment (start 134.55 94.99) (end 136.56 94.99) (width 0.1778) (layer F.Cu) (net 6))
   (segment (start 136.56 94.99) (end 136.62 94.93) (width 0.1778) (layer F.Cu) (net 6))
   (zone (net 2) (net_name GND) (layer B.Cu) (hatch edge 0.508)
-    (connect_pads (clearance 0.508))
+    (connect_pads (clearance 0.254))
     (min_thickness 0.254)
     (fill yes (arc_segments 16) (thermal_gap 0.508) (thermal_bridge_width 0.508))
