File: fx2_tube_cartridge_adapter/pcb/fx2_tube_cartridge_adapter.kicad_pcb (KiCad board)
At the start: 2 copper layers, 66.5 x 76.5 mm, 41 parts, among them U1 MCP1700T-3302E/MB

Commit message: fx2_tube_cartridge_adapter ready for fab
Parts:
- added EXTPWR: ext pwr, Pin_Headers:Pin_Header_Straight_1x03_Pitch2.54mm, F.Cu at (55.5, 62.8)
- added LEADS: Options, Pin_Headers:Pin_Header_Straight_2x04_Pitch2.54mm, F.Cu at (93.1, 19.9)
- added R6: 1k, Resistors_SMD:R_0805_HandSoldering, F.Cu at (81.0, 23.2)
- added staple_single21: , myelin-kicad:via_single, F.Cu at (108.5, 14.2)
- added staple_single22: , myelin-kicad:via_single, F.Cu at (49.3, 14.7)
- added staple_single23: , myelin-kicad:via_single, F.Cu at (93.8, 66.4)
- added staple_single24: , myelin-kicad:via_single, F.Cu at (92.5, 67.6)
- added staple_single25: , myelin-kicad:via_single, F.Cu at (90.9, 69.2)
- added staple_single26: , myelin-kicad:via_single, F.Cu at (92.4, 70.7)
- added staple_single27: , myelin-kicad:via_single, F.Cu at (76.7, 68.4)
- added staple_single28: , myelin-kicad:via_single, F.Cu at (91.7, 30.2)
- added staple_single29: , myelin-kicad:via_single, F.Cu at (67.5, 40.4)
- added staple_single30: , myelin-kicad:via_single, F.Cu at (85.4, 40.3)
- added staple_single31: , myelin-kicad:via_single, F.Cu at (95.7, 46.8)
- added staple_single32: , myelin-kicad:via_single, F.Cu at (98.2, 42.9)
- R5: footprint Resistors_SMD:R_0805 -> Resistors_SMD:R_0805_HandSoldering
- moved staple_single17 95.9 mm to (67.1, 21.6)
- moved staple_single18 95.5 mm to (69.3, 21.5)
- moved staple_single19 95.1 mm to (71.6, 21.6)
- moved staple_single20 94.8 mm to (74.5, 21.6)
- moved staple_single15 56.3 mm to (76.3, 60.1)
- moved staple_single14 53.6 mm to (82.2, 62.2)
- moved staple_single16 49.8 mm to (49.4, 81.2)
- moved staple_single12 48.5 mm to (74.5, 68.5)
- moved staple_single13 47.5 mm to (82.7, 68.3)
- moved D1 28.1 mm to (57.8, 40.4), turned to 0 degrees
- moved R5 19.6 mm to (57.9, 44.8), turned to 0 degrees
- moved PIPWR 15.4 mm to (49.0, 58.7), turned to 0 degrees
- moved R4 14.6 mm to (81.0, 25.3)
- moved R3 14.6 mm to (81.0, 27.5)
- moved FX2PWR 14.1 mm to (49.2, 67.1), turned to 0 degrees
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- renumbered CONN to FX2
Connections:
- CART pad A11: cpu_READY -> elk_READY_master_RnW
- FX2 pad L2: tube_nRST -> cpu_nRST
- FX2 pad L7: (no net) -> analyzer_RDY0
- FX2 pad L8: cpu_CLK_jumper -> tube_CLK_jumper
- FX2 pad R3: cpu_READY -> analyzer_PD2_READY
- FX2 pad R5: tube_RnW -> analyzer_PD0_RnW
- PI1 pad 1: (no net) -> 3V3_PI
- PI1 pad 17: 3V3_PI -> (no net)
- PI1 pad 2: 5V_PI -> (no net)
- PI1 pad 4: 5V_PI -> (no net)
- R1 pad 2: 3V3 -> 3V3_FX2
- R2 pad 2: 3V3 -> 3V3_FX2
- R4 pad 2: 3V3 -> 3V3_FX2
- R5 pad 1: 3V3 -> 3V3_PI
Routing:
- net cpu_nRST: track 21.7 -> 127.7 mm
- net elk_READY_master_RnW: track 0.00 -> 96.3 mm, vias 0 -> 4
- net cpu_READY: track 69.7 -> 0.00 mm, vias 3 -> 0
- net 3V3: track 14.5 -> 77.9 mm, vias 0 -> 2
- net tube_nRST: track 69.2 -> 11.2 mm
- net analyzer_PD0_RnW: track 0.00 -> 52.5 mm, vias 0 -> 1
- net tube_RnW: track 35.1 -> 78.9 mm, vias 2 -> 3
- net cpu_SYNC: track 0.00 -> 36.8 mm
- net 3V3_FX2: track 51.0 -> 87.7 mm, vias 0 -> 1
- net analyzer_PD2_READY: track 0.00 -> 36.0 mm, vias 0 -> 1
- net tube_CLK: track 19.2 -> 48.8 mm
- net analyzer_PA2: track 0.00 -> 22.2 mm, vias 0 -> 2
- net analyzer_PA4: track 0.00 -> 18.7 mm, vias 0 -> 2
- net cpld_TDI: track 0.00 -> 17.5 mm
- net cpld_TCK: track 0.00 -> 16.8 mm
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Other:
- board size 66.5 x 76.5 mm -> 66.5 x 74.5 mm
- board text added: "/NMI"
- board text added: "0 3 5"
- board text added: "Bridge for synchronous capture"
- board text added: "Bridge on Elk/BBC"
- board text added: "Bridge on Master"
- board text added: "GND Tx Rx"
- board text added: "READY"
- board text added: "SYNC"
- board text removed: "- check all TODO items in python netlist"

Commit message: r2: Added a bunch of TODOs, implemented some, made silkscreen more assembly-friendly
Other:
- board text added: "Electron cartridge / BBC Tube adapter r2 for FX2 logic analyzer + decode6502 http://myelin.nz/acorn/fx2tube Copyright 2017 Google LLC Designed by Phillip Pearson"
- board text removed: "Electron cartridge / BBC Tube adapter for FX2 logic analyzer + decode6502 http://myelin.nz/acorn/fx2tube Copyright 2017 Google LLC Designed by Phillip Pearson"
Changed lines of the file:
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@@
     (links 190)
     (no_connects 0)
-    (area 42.40022 2.4384 116.232941 99.011741)
+    (area 45.699999 10.949999 112.300001 85.550001)
     (thickness 1.6)
-    (drawings 25)
+    (drawings 31)
     (tracks 880)
     (zones 0)
@@
       (effects (font (size 1 1) (thickness 0.15)))
     )
-    (fp_text value 1k (at 0 1.75) (layer F.Fab)
+    (fp_text value 1k (at 6.39952 0.0635) (layer F.SilkS)
       (effects (font (size 1 1) (thickness 0.15)))
     )
@@
       (effects (font (size 1 1) (thickness 0.15)))
     )
-    (fp_text value 1k (at 0 1.75) (layer F.Fab)
+    (fp_text value 1k (at 6.3665 -0.13716) (layer F.SilkS)
       (effects (font (size 1 1) (thickness 0.15)))
     )
@@
       (effects (font (size 1 1) (thickness 0.15)))
     )
-    (fp_text value 1k (at 0 1.75) (layer F.Fab)
+    (fp_text value 1k (at 6.39952 -0.08382) (layer F.SilkS)
       (effects (font (size 1 1) (thickness 0.15)))
     )
@@
       (effects (font (size 1 1) (thickness 0.15)))
     )
-    (fp_text value 1k (at 0 1.75) (layer F.Fab)
+    (fp_text value 1k (at 6.38428 0.33782) (layer F.SilkS)
       (effects (font (size 1 1) (thickness 0.15)))
     )
@@
     (tags "capacitor 0805")
     (attr smd)
-    (fp_text reference C4 (at 3.15468 -0.59182 270) (layer F.SilkS)
-      (effects (font (size 1 1) (thickness 0.15)))
-    )
-    (fp_text value 1u (at 0 1.75 90) (layer F.Fab)
+    (fp_text reference C4 (at 2.99564 -0.02818 360) (layer F.SilkS)
+      (effects (font (size 1 1) (thickness 0.15)))
+    )
+    (fp_text value 1u (at 0.97564 1.92182 180) (layer F.SilkS)
       (effects (font (size 1 1) (thickness 0.15)))
     )
@@
     (tags "capacitor 0805")
     (attr smd)
-    (fp_text reference C5 (at -3.09372 0.3937 270) (layer F.SilkS)
-      (effects (font (size 1 1) (thickness 0.15)))
-    )
-    (fp_text value 1u (at 0 1.75 270) (layer F.Fab)
+    (fp_text reference C5 (at -3.02294 -0.01034 360) (layer F.SilkS)
+      (effects (font (size 1 1) (thickness 0.15)))
+    )
+    (fp_text value 1u (at 0.91706 -4.09034 360) (layer F.SilkS)
       (effects (font (size 1 1) (thickness 0.15)))
     )
@@
     (tags "capacitor 0805")
     (attr smd)
-    (fp_text reference C1 (at -2.67684 -1.02108 270) (layer F.SilkS)
-      (effects (font (size 1 1) (thickness 0.15)))
-    )
-    (fp_text value 100n (at 0 1.75 90) (layer F.Fab)
+    (fp_text reference C1 (at 2.09304 -0.05254 360) (layer F.SilkS)
+      (effects (font (size 1 1) (thickness 0.15)))
+    )
+    (fp_text value 100n (at 0.25304 1.33746 270) (layer F.SilkS)
       (effects (font (size 1 1) (thickness 0.15)))
     )
@@
       (effects (font (size 1 1) (thickness 0.15)))
     )
-    (fp_text value 100n (at 0 1.75 180) (layer F.Fab)
+    (fp_text value 100n (at 3.68422 0.14286 180) (layer F.SilkS)
       (effects (font (size 1 1) (thickness 0.15)))
     )
@@
     (tags "capacitor 0805")
     (attr smd)
-    (fp_text reference C3 (at 0.71374 -1.41986 90) (layer F.SilkS)
-      (effects (font (size 1 1) (thickness 0.15)))
-    )
-    (fp_text value 1u (at 0 1.75 90) (layer F.Fab)
+    (fp_text reference C3 (at 0.90256 -1.97786 180) (layer F.SilkS)
+      (effects (font (size 1 1) (thickness 0.15)))
+    )
+    (fp_text value 1u (at -0.52744 -1.97786 180) (layer F.SilkS)
       (effects (font (size 1 1) (thickness 0.15)))
     )
@@
     (tags SOD-323)
     (attr smd)
-    (fp_text reference D1 (at 0 -1.85) (layer F.SilkS)
+    (fp_text reference D1 (at 0.00278 -3.3087) (layer F.SilkS)
       (effects (font (size 1 1) (thickness 0.15)))
     )
@@
       (effects (font (size 1 1) (thickness 0.15)))
     )
-    (fp_text value 1k (at 0 1.75) (layer F.Fab)
+    (fp_text value 1k (at 6.3411 0.10668) (layer F.SilkS)
       (effects (font (size 1 1) (thickness 0.15)))
     )
@@
       (effects (font (size 1 1) (thickness 0.15)))
     )
-    (fp_text value 10k (at 0 1.75) (layer F.Fab)
+    (fp_text value 10k (at 0 1.75) (layer F.SilkS)
       (effects (font (size 1 1) (thickness 0.15)))
     )
@@
     )
   )
+  (gr_line (start 57.48 38.56) (end 56.98 38.56) (layer F.SilkS) (width 0.2))
+  (gr_line (start 57.48 38.06) (end 57.48 39.06) (layer F.SilkS) (width 0.2))
+  (gr_line (start 57.48 38.56) (end 57.98 38.06) (layer F.SilkS) (width 0.2))
+  (gr_line (start 57.98 39.06) (end 57.48 38.56) (layer F.SilkS) (width 0.2))
+  (gr_line (start 57.98 38.06) (end 57.98 39.06) (layer F.SilkS) (width 0.2))
+  (gr_line (start 58.48 38.56) (end 57.98 38.56) (layer F.SilkS) (width 0.2))
   (gr_line (start 90.17 20.701) (end 91.059 20.701) (layer F.SilkS) (width 0.2))
   (gr_line (start 90.17 16.51) (end 90.17 20.701) (layer F.SilkS) (width 0.2))
@@
   (gr_line (start 107.25 85.5) (end 112.25 80.5) (layer Edge.Cuts) (width 0.1))
   (gr_line (start 112.25 16) (end 112.25 80.5) (layer Edge.Cuts) (width 0.1))
-  (gr_text "Electron cartridge / BBC Tube adapter\nfor FX2 logic analyzer + decode6502\n\nhttp://myelin.nz/acorn/fx2tube\n\nCopyright 2017 Google LLC\nDesigned by Phillip Pearson" (at 77.0128 64.17564) (layer B.SilkS)
+  (gr_text "Electron cartridge / BBC Tube adapter r2\nfor FX2 logic analyzer + decode6502\n\nhttp://myelin.nz/acorn/fx2tube\n\nCopyright 2017 Google LLC\nDesigned by Phillip Pearson" (at 77.0128 64.17564) (layer B.SilkS)
     (effects (font (size 1 1) (thickness 0.2)) (justify mirror))
   )
