File: a3000_rom_emulator/a5000_adapter_pcb/a5000_adapter.kicad_pcb (KiCad board)
At the start: 2 copper layers, 43.2 x 83.8 mm, 8 parts

Commit message: Wired up adapter, and brought out A21 for easy connection to arcflash board
Parts:
- added A21: , Connector_PinHeader_2.54mm:PinHeader_1x01_P2.54mm_Vertical, F.Cu at (139.7, 61.0)
Connections:
- A3KROM1 pad 16: rom1_pin16 -> GND
- A3KROM1 pad 32: rom1_pin32 -> rom_5V
- A3KROM2 pad 16: rom2_pin16 -> GND
- A3KROM2 pad 32: rom2_pin32 -> rom_5V
- A3KROM3 pad 16: rom3_pin16 -> GND
- A3KROM3 pad 32: rom3_pin32 -> rom_5V
- A3KROM4 pad 16: rom4_pin16 -> GND
- A3KROM4 pad 32: rom4_pin32 -> rom_5V
- A5KROM1 pad 16: rom1_pin16 -> GND
- A5KROM1 pad 32: rom1_pin32 -> rom_5V
- A5KROM2 pad 16: rom2_pin16 -> GND
- A5KROM2 pad 32: rom2_pin32 -> rom_5V
- A5KROM3 pad 16: rom3_pin16 -> GND
- A5KROM3 pad 32: rom3_pin32 -> rom_5V
- A5KROM4 pad 16: rom4_pin16 -> GND
- A5KROM4 pad 32: rom4_pin32 -> rom_5V
Routing:
- net rom4_pin31: track 0.00 -> 13.8 mm
- net rom1_pin1: track 5.96 -> 19.5 mm
- net rom4_pin28: track 0.00 -> 13.6 mm
- net rom4_pin24: track 0.00 -> 13.6 mm
- net rom4_pin17: track 0.00 -> 13.6 mm
- net rom4_pin23: track 0.00 -> 13.6 mm
- net rom4_pin20: track 0.00 -> 13.6 mm
- net rom_5V: track 0.00 -> 13.6 mm
- net rom4_pin32: track 13.6 -> 0.00 mm
- net rom4_pin30: track 0.00 -> 13.6 mm
- net rom4_pin29: track 0.00 -> 13.6 mm
- net rom4_pin27: track 0.00 -> 13.6 mm
- net rom4_pin26: track 0.00 -> 13.6 mm
- net rom4_pin22: track 0.00 -> 13.6 mm
- net rom4_pin21: track 0.00 -> 13.6 mm
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- added copper zone on B.Cu, net GND
- added copper zone on F.Cu, net rom_5V

Commit message: v1 ready to go to JLC
Other:
- board text added: "THIS SIDE UP! * Arcflash byte order 3210 *"
- board text removed: "-- THIS SIDE FACES UP --"
Changed lines of the file:
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@@
     (effects (font (size 1 1) (thickness 0.2)) (justify mirror))
   )
-  (gr_text "-- THIS SIDE FACES UP --" (at 158.75 60.96) (layer F.SilkS)
+  (gr_text "THIS SIDE UP!  * Arcflash byte order 3210 *" (at 162.55 60.89) (layer F.SilkS)
     (effects (font (size 1 1) (thickness 0.2)))
   )
@@
   (segment (start 156.413299 112.826701) (end 156.413299 123.393299) (width 0.1778) (layer B.Cu) (net 109))
   (segment (start 157.48 111.76) (end 156.413299 112.826701) (width 0.1778) (layer B.Cu) (net 109))
-  (segment (start 138.900001 123.660001) (end 139.7 124.46) (width 0.1778) (layer B.Cu) (net 122))
-  (segment (start 138.633299 123.393299) (end 138.900001 123.660001) (width 0.1778) (layer B.Cu) (net 122))
-  (segment (start 138.633299 112.826701) (end 138.633299 123.393299) (width 0.1778) (layer B.Cu) (net 122))
-  (segment (start 139.7 111.76) (end 138.633299 112.826701) (width 0.1778) (layer B.Cu) (net 122))
   (segment (start 159.220001 123.660001) (end 160.02 124.46) (width 0.1778) (layer B.Cu) (net 110))
   (segment (start 158.953299 112.826701) (end 158.953299 123.393299) (width 0.1778) (layer B.Cu) (net 110))
@@
   (segment (start 172.72 127) (end 172.72 139.7) (width 0.1778) (layer F.Cu) (net 119))
   (segment (start 170.18 139.7) (end 170.18 127) (width 0.1778) (layer F.Cu) (net 120))
+  (segment (start 138.900001 123.660001) (end 139.7 124.46) (width 0.1778) (layer B.Cu) (net 122))
+  (segment (start 138.633299 123.393299) (end 138.900001 123.660001) (width 0.1778) (layer B.Cu) (net 122))
+  (segment (start 138.633299 112.826701) (end 138.633299 123.393299) (width 0.1778) (layer B.Cu) (net 122))
+  (segment (start 139.7 111.76) (end 138.633299 112.826701) (width 0.1778) (layer B.Cu) (net 122))
   (zone (net 122) (net_name rom_5V) (layer F.Cu) (hatch edge 0.508)
     (connect_pads (clearance 0.1778))
