File: econet_from_scratch/pcb/econet_standalone.kicad_pcb (KiCad board)
At the start: 2 copper layers, 48.5 x 48 mm, 72 parts, among them U1 Econet, U2 SN65C1168, U3 LM319, U4 XC9572XL, U5 MCP1700T-3302E/MB

Commit message: Some unpushed changes from months ago -- progress on USB Econet
Connections:
- net PA08 renamed serial_mcu_to_cpld
- net PA09 renamed serial_buffer_empty
- net PA10 renamed outputting_frame
- net PA11 renamed mcu_is_transmitting
- net PA14 renamed serial_cpld_to_mcu
- net PA15 renamed clock_24m
- net PA16 renamed drive_econet_clock
- net PA17 renamed econet_clock_from_mcu
- net mcu_RXD renamed mcu_debug_RXD
- net mcu_TXD renamed mcu_debug_TXD
