File: arc_keyboard_to_a3000/pcb/arc_keyboard_to_a3000.kicad_pcb (KiCad board)
At the start: 2 copper layers, 17.1 x 20.3 mm, 2 parts

Commit message: Arc keyboard USB interface
Other:
- board text added: "KIN = Krx* = data from keyboard KOUT = Ktx* = data to keyboard"
Changed lines of the file:
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@@
   (general
     (thickness 1.6)
-    (drawings 6)
+    (drawings 7)
     (tracks 28)
     (zones 0)
@@
       (net 5 KOUT))
   )
+  (gr_text "KIN = Krx* = data from keyboard\nKOUT = Ktx* = data to keyboard" (at 137.93724 106.95432) (layer Cmts.User)
+    (effects (font (size 1 1) (thickness 0.2)) (justify left))
+  )
   (gr_text "pp@myelin.nz\narc_keyboard_to_a3000" (at 129.14376 101.47808 90) (layer B.SilkS)
