File: elk_pi_tube_direct/pcb/elk_pi_tube_direct.kicad_pcb (KiCad board)
At the start: 2 copper layers, 77 x 59.5 mm, 10 parts

Commit message: Added some notes on how to build an SD card adapter for the Electron
Routing:
- net cpld_TCK: track 17.6 -> 18.4 mm
- net elk_D2: track 33.2 -> 32.4 mm
- net tube_A1: track 27.6 -> 28.2 mm
Other:
- board text added: "A 5V 5V TX RX RnW GND D5 D6 GND D7 D0 PHI0"
- board text added: "A B"
- board text added: "Acorn Electron PiTubeDirect Interface v2"
- board text added: "Acorn Electron PiTubeDirect Interface v2 Phillip Pearson <pp@myelin.nz> Copyright 2017 Google Inc"
- board text added: "B 3V A1 A2 /RST GND /TUBE A0 D4 3V3 D2 D1 D3 GND"
- board text removed: "Acorn Electron PiTubeDirect Interface"
- board text removed: "Acorn Electron PiTubeDirect Interface Phillip Pearson <pp@myelin.nz> Copyright 2017 Google Inc"
